File: RFM69W-V1.0.sch (EAGLE design)
At the start: 14 parts, among them J1 NRF connector, J2 SD card

Commit message: Cosmetic update
Parts:
- removed LED1: RED, dp_devices:LED-0805
- removed LED2: GREEN, dp_devices:LED-0805
- removed LED3: YELLOW, dp_devices:LED-0805
- added U$2, U$3, U$4: LED0805-LARGE, _c2h:LED0805-LARGE
- C1: device resistor:C-EUC0805K -> _c2h:CAP0805-CAP
- C2: device resistor:C-EUC0805 -> _c2h:CAP0805-CAP
- R1, R2, R3, R4: device resistor:R-US_M0805 -> _c2h:RESISTOR0805-RES
Connections:
- net CE: now also U$2.MINUS; no longer LED1.C
- net CSN: now also U$3.MINUS; no longer LED2.C
- net IRQ: now also U$4.MINUS; no longer LED3.C
- net N$2: now also U$2.PLUS; no longer LED1.A
- net N$3: now also U$3.PLUS; no longer LED2.A
- net N$5: now also U$4.PLUS; no longer LED3.A
Other:
- note added: "Only used for future mode of RFM69 if you use this pin you can't use SD nor SPI flash (share the same pin)"
- note added: "RFM69(H)W Breakout Board with MicroSD support and Flash SPI eeprom see http://hallard.me"
- note removed: "R4 only used for OOK mode of RFM12B if you use OOK mode you can't use SD nor SPI flash (share the same pin)"
- note removed: "RFM69HW Breakout Board with MicroSD support and Flash SPI eeprom see http://hallard.me"
- moved on the sheet: C1, C2
